Commit message: bravo7_no_ee_v2 modification finished and tested

File: robots/bravo7_description/urdf/bravo7_no_ee_v2.urdf (robot description, URDF)
Before this commit: robot bravo7_no_ee_v2, 10 links, 9 joints
Links:
- removed link force_torque_sensor
- link link2: mass 1.55 -> 1.62
- link link3: mass 1.14 -> 2.12
- link link4: mass 1.14 -> 1.33
- link link5: mass 1.03 -> 1.33
- link link6: mass 0.333 -> 0.97
- link link7: mass 1.04 -> 1.09
Joints:
- removed joint FT_fixed_1
- joint contact_point_joint: parent force_torque_sensor -> link7
- joint joint1: axis 0 0 1 -> 0 0 -1; origin xyz=0.0665 0 0.078 rpy=3.141592654 0 0 -> xyz=0.0665 0 0.078 rpy=0 0 0
- joint joint2: origin xyz=-0.046 0 -0.0674 rpy=3.141592654 0 0 -> xyz=-0.046 0 0.0674 rpy=0 0 0
- joint joint4: axis 0 0 1 -> 0 0 -1; origin xyz=0.0408 0 0.09695 rpy=3.141592654 0 0 -> xyz=0.0408 0 0.09695 rpy=0 0 0
- joint joint5: origin xyz=-0.0408 0 -0.063 rpy=3.141592654 0 0 -> xyz=-0.0408 0 0.063 rpy=0 0 0
- joint joint6: axis 0 0 1 -> 0 0 -1; origin xyz=-0.0408 0 -0.14863 rpy=0 3.14159 0 -> xyz=-0.0408 0 -0.08863 rpy=0 3.14159 0

Commit message: bravo7_no_ee_v2.urdf ready with correct masses and inertias

File: robots/bravo7_description/urdf/bravo7_no_ee_v2.urdf (robot description, URDF)
Before this commit: robot bravo7_no_ee_v2, 9 links, 8 joints
Joints:
- joint joint1: axis 0 0 -1 -> 0 0 1; origin xyz=0.0665 0 0.078 rpy=0 0 0 -> xyz=0.0665 0 0.078 rpy=3.141592654 0 0
- joint joint2: origin xyz=-0.046 0 0.0674 rpy=0 0 0 -> xyz=-0.046 0 -0.0674 rpy=3.141592654 0 0
- joint joint4: axis 0 0 -1 -> 0 0 1; origin xyz=0.0408 0 0.09695 rpy=0 0 0 -> xyz=0.0408 0 0.09695 rpy=3.141592654 0 0
- joint joint5: origin xyz=-0.0408 0 0.063 rpy=0 0 0 -> xyz=-0.0408 0 -0.063 rpy=3.141592654 0 0
- joint joint6: axis 0 0 -1 -> 0 0 1
