Commit message: Adding urdf with collision models defined as cylinders

File: robots/bravo7_description/urdf/bravo7_identification.urdf (robot description, URDF)
Before this commit: robot bravo7_identification, 9 links, 8 joints
Links:
- link end_effector_ball: geometry collision cylinder length=0.09 radius=0.05; visual mesh filename=package://example-robot-data/robots/bravo7_description/mesh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
- link link1: geometry collision cylinder length=0.085 radius=0.074; visual mesh filename=package://example-robot-data/robots/bravo7_description/mesh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
- link link2: geometry collision cylinder length=0.11 radius=0.074; visual mesh filename=package://example-robot-data/robots/bravo7_description/mesh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
- link link3: geometry collision cylinder length=0.3 radius=0.06; visual mesh filename=package://example-robot-data/robots/bravo7_description/mesh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
- link link4: geometry collision cylinder length=0.12 radius=0.055; visual mesh filename=package://example-robot-data/robots/bravo7_description/mesh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
- link link5: geometry collision cylinder length=0.1 radius=0.055; visual mesh filename=package://example-robot-data/robots/bravo7_description/mesh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
- link link6: geometry collision cylinder length=0.1 radius=0.055; visual mesh filename=package://example-robot-data/robots/bravo7_description/mesh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
- link link7: geometry collision cylinder length=0.12 radius=0.05; visual mesh filename=package://example-robot-data/robots/bravo7_description/mesh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

Commit message: Adding bravo identification with revolute joints

File: robots/bravo7_description/urdf/bravo7_identification.urdf (robot description, URDF)
Before this commit: robot bravo7_identification, 9 links, 8 joints
Links:
- added link world
Joints:
- added joint base_static_joint: type fixed, parent world, child link1, origin xyz=0 0 0 rpy=0 -1.5708  0
